File: macropad-v2_0_0/macropad-v2_0_0.sch (KiCad schematic (older format))
At the start: 13 parts, among them SW1 SW_Push, SW2 SW_Push, SW3 SW_Push, SW4 SW_Push, SW5 SW_Push, SW6 SW_Push, U1 ProMicro

Commit message: Adding README
Parts:
- added J1: Conn_01x04_Male, Connector_PinHeader_2.54mm:PinHeader_1x04_P2.54mm_Vertical, symbol Connector:Conn_01x04_Male
- added SW7: Rotary_Encoder_Switch, Gauntface:ACZ11BRXE, symbol Device:Rotary_Encoder_Switch
- U1: symbol promicro:ProMicro -> macropad-v2_0_0-rescue:ProMicro-promicro
Connections:
- net at U1.17 (F7): now also SW7.S2
- net at U1.18 (F6): now also SW7.B
- net at U1.19 (F5): now also SW7.C
- net at U1.20 (F4): now also SW7.A
- net GND: now reaches U1.23 (GND)
- net GND: now also J1.4 (Pin_4), SW7.S1
- net at U1.5 (SDA): now also J1.1 (Pin_1)
- net at U1.6 (SCL): now also J1.2 (Pin_2)
- new net VCC: J1.3 (Pin_3)
Changed lines of the file:
@@
 $EndComp
 $Comp
-L promicro:ProMicro U1
+L macropad-v2_0_0-rescue:ProMicro-promicro U1
 U 1 1 604F2D20
 P 5350 3500
@@
 Text Label 4650 3550 2    50   ~ 0
 Col_0
+$Comp
+L Device:Rotary_Encoder_Switch SW7
+U 1 1 6057EBC9
+P 6950 3300
+F 0 "SW7" H 6950 3667 50  0000 C CNN
+F 1 "Rotary_Encoder_Switch" H 6950 3576 50  0000 C CNN
+F 2 "Gauntface:ACZ11BRXE" H 6800 3460 50  0001 C CNN
+F 3 "~" H 6950 3560 50  0001 C CNN
+	1    6950 3300
+	1    0    0    -1
+$EndComp
+Wire Wire Line
+	6050 3150 6650 3150
+Wire Wire Line
+	6650 3150 6650 3200
+Wire Wire Line
+	6050 3250 6650 3250
+Wire Wire Line
+	6650 3250 6650 3300
+Wire Wire Line
+	6050 3350 6650 3350
+Wire Wire Line
+	6650 3350 6650 3400
+Wire Wire Line
+	6050 3450 7250 3450
+Wire Wire Line
+	7250 3450 7250 3400
+$Comp
+L power:GND #PWR0101
+U 1 1 60581374
+P 7450 3200
+F 0 "#PWR0101" H 7450 2950 50  0001 C CNN
+F 1 "GND" H 7455 3027 50  0000 C CNN
+F 2 "" H 7450 3200 50  0001 C CNN
+F 3 "" H 7450 3200 50  0001 C CNN
+	1    7450 3200
+	1    0    0    -1
+$EndComp
+Wire Wire Line
+	7450 3200 7250 3200
+$Comp
+L Connector:Conn_01x04_Male J1
+U 1 1 60581994
+P 3700 3250
+F 0 "J1" H 3808 3531 50  0000 C CNN
+F 1 "Conn_01x04_Male" H 3808 3440 50  0000 C CNN
+F 2 "Connector_PinHeader_2.54mm:PinHeader_1x04_P2.54mm_Vertical" H 3700 3250 50  0001 C CNN
+F 3 "~" H 3700 3250 50  0001 C CNN
+	1    3700 3250
+	1    0    0    -1
+$EndComp
+Wire Wire Line
+	3900 3150 4650 3150
+Wire Wire Line
+	4650 3250 3900 3250
+$Comp
+L power:VCC #PWR02
+U 1 1 605842C8
+P 4250 3350
+F 0 "#PWR02" H 4250 3200 50  0001 C CNN
+F 1 "VCC" H 4265 3523 50  0000 C CNN
+F 2 "" H 4250 3350 50  0001 C CNN
+F 3 "" H 4250 3350 50  0001 C CNN
+	1    4250 3350
+	-1   0    0    1
+$EndComp
+$Comp
+L power:GND #PWR01
+U 1 1 60584EA4
+P 4050 3450
+F 0 "#PWR01" H 4050 3200 50  0001 C CNN
+F 1 "GND" H 4055 3277 50  0000 C CNN
+F 2 "" H 4050 3450 50  0001 C CNN
+F 3 "" H 4050 3450 50  0001 C CNN
+	1    4050 3450
+	1    0    0    -1
+$EndComp
+Wire Wire Line
+	3900 3350 4250 3350
+Wire Wire Line
+	3900 3450 4050 3450
+$Comp
+L power:GND #PWR03
+U 1 1 60587943
+P 6300 2850
+F 0 "#PWR03" H 6300 2600 50  0001 C CNN
+F 1 "GND" V 6305 2722 50  0000 R CNN
+F 2 "" H 6300 2850 50  0001 C CNN
+F 3 "" H 6300 2850 50  0001 C CNN
+	1    6300 2850
+	0    -1   -1   0
+$EndComp
+Wire Wire Line
+	6050 2850 6300 2850
 $EndSCHEMATC

Commit message: Started coding up the keyboard matrix and finished v2
Parts:
- removed U1: ProMicro, promicro:ProMicro, symbol macropad-v2_0_0-rescue:ProMicro-promicro
- added D7, D8: D, Diode_THT:D_A-405_P7.62mm_Horizontal, symbol Device:D
- added SW8: Layer_Btn, Button_1825910-6:SW_1825910-6-4, symbol 1825910-6:1825910-6
- added SW9: Reset_Btn, Button_1825910-6:SW_1825910-6-4, symbol 1825910-6:1825910-6
- added U1: ProMicro, promicro:ProMicro, symbol promicro:ProMicro
- J1: footprint Connector_PinHeader_2.54mm:PinHeader_1x04_P2.54mm_Vertical -> Gauntface:Screen_38x12mm_JMD0_91_a
- SW1: value SW_Push -> Key_1; footprint Switch_Keyboard_Cherry_MX:SW_Cherry_MX_PCB -> Switch_Keyboard_Kailh:SW_Hotswap_Kailh
- SW2: value SW_Push -> Key_2; footprint Switch_Keyboard_Cherry_MX:SW_Cherry_MX_PCB -> Switch_Keyboard_Kailh:SW_Hotswap_Kailh
- SW3: value SW_Push -> Key_3; footprint Switch_Keyboard_Cherry_MX:SW_Cherry_MX_PCB -> Switch_Keyboard_Kailh:SW_Hotswap_Kailh
- SW4: value SW_Push -> Key_4; footprint Switch_Keyboard_Cherry_MX:SW_Cherry_MX_PCB -> Switch_Keyboard_Kailh:SW_Hotswap_Kailh
- SW5: value SW_Push -> Key_5; footprint Switch_Keyboard_Cherry_MX:SW_Cherry_MX_PCB -> Switch_Keyboard_Kailh:SW_Hotswap_Kailh
- SW6: value SW_Push -> Key_6; footprint Switch_Keyboard_Cherry_MX:SW_Cherry_MX_PCB -> Switch_Keyboard_Kailh:SW_Hotswap_Kailh
Connections:
- net labels added: Encoder_S1, Encoder_S2, Row_Extra
- wire segments 29 -> 46
- no-connect marks 0 -> 9
Other:
- moved on the sheet: D1, D2, D3, D4, D5, D6, J1, SW1, SW2, SW3, SW4, SW5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
