File: macropad-v2_0_1/macropad-v2_0_1.sch (KiCad schematic (older format))
At the start: 19 parts, among them J1 Conn_01x04_Male, SW1 Key_1, SW2 Key_2, SW3 Key_3, SW4 Key_4, SW5 Key_5, SW6 Key_6, SW7 Rotary_Encoder_Switch, SW8 Layer_Btn, SW9 Reset_Btn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

Commit message: Adding paths to schematic
Parts:
- SW8, SW9: symbol 1825910-6:1825910-6 -> macropad-v2_0_1-rescue:1825910-6-1825910-6
- U1: symbol promicro:ProMicro -> macropad-v2_0_1-rescue:ProMicro-promicro
Connections:
- net Col_0: now also U1.14 (16); no longer U1.10 (7)
- net Col_1: now also U1.13 (10); no longer U1.8 (5)
- net Col_2: now also U1.15 (14); no longer U1.7 (4)
- net Row_Extra: now also U1.16 (15); no longer U1.9 (6)
- net Encoder_A: now reaches SW7.A
- net Encoder_A: now also U1.8 (5); no longer U1.15 (14)
- net Encoder_B: now reaches SW7.B
- net Encoder_B: now also U1.9 (6); no longer U1.16 (15)
Other:
- moved on the sheet: SW7
Changed lines of the file:
@@
 L Device:Rotary_Encoder_Switch SW7
 U 1 1 6057EBC9
-P 6950 3650
-F 0 "SW7" H 6950 4017 50  0000 C CNN
-F 1 "Rotary_Encoder_Switch" H 6950 3926 50  0000 C CNN
-F 2 "Gauntface:ACZ11BRXE" H 6800 3810 50  0001 C CNN
-F 3 "~" H 6950 3910 50  0001 C CNN
-	1    6950 3650
+P 6000 5200
+F 0 "SW7" H 6000 5567 50  0000 C CNN
+F 1 "Rotary_Encoder_Switch" H 6000 5476 50  0000 C CNN
+F 2 "Gauntface:ACZ11BRXE" H 5850 5360 50  0001 C CNN
+F 3 "~" H 6000 5460 50  0001 C CNN
+	1    6000 5200
 	1    0    0    -1
 $EndComp
@@
 	1650 6300 1900 6300
 Connection ~ 1900 6300
-Text GLabel 4650 3750 0    50   Input ~ 0
-Row_0
-Text GLabel 4650 3850 0    50   Input ~ 0
-Row_1
-Text GLabel 4650 3550 0    50   Input ~ 0
+Text GLabel 6050 3550 2    50   Input ~ 0
 Row_Extra
-Text GLabel 4650 3650 0    50   Input ~ 0
+Text GLabel 6050 3750 2    50   Input ~ 0
 Col_0
-Text GLabel 4650 3450 0    50   Input ~ 0
+Text GLabel 6050 3850 2    50   Input ~ 0
 Col_1
-Text GLabel 4650 3350 0    50   Input ~ 0
+Text GLabel 6050 3650 2    50   Input ~ 0
 Col_2
-Text GLabel 7250 3550 2    50   Input ~ 0
+Text GLabel 6300 5100 2    50   Input ~ 0
 Encoder_S1
-Text GLabel 7250 3750 2    50   Input ~ 0
+Text GLabel 6300 5300 2    50   Input ~ 0
 Encoder_S2
 $Comp
@@
 $EndComp
 $Comp
-L promicro:ProMicro U1
+L macropad-v2_0_1-rescue:ProMicro-promicro U1
 U 1 1 6077E1C9
 P 5350 3500
@@
 L power:GND #PWR07
 U 1 1 60785B0E
-P 6650 3650
-F 0 "#PWR07" H 6650 3400 50  0001 C CNN
-F 1 "GND" V 6655 3522 50  0000 R CNN
-F 2 "" H 6650 3650 50  0001 C CNN
-F 3 "" H 6650 3650 50  0001 C CNN
-	1    6650 3650
+P 5700 5200
+F 0 "#PWR07" H 5700 4950 50  0001 C CNN
+F 1 "GND" V 5705 5072 50  0000 R CNN
+F 2 "" H 5700 5200 50  0001 C CNN
+F 3 "" H 5700 5200 50  0001 C CNN
+	1    5700 5200
 	0    1    1    0
 $EndComp
@@
 NoConn ~ 6050 3250
 NoConn ~ 6050 3150
-NoConn ~ 6050 3750
-NoConn ~ 6050 3850
 Wire Wire Line
 	6050 2950 6500 2950
@@
 $EndComp
 $Comp
-L 1825910-6:1825910-6 SW9
+L macropad-v2_0_1-rescue:1825910-6-1825910-6 SW9
 U 1 1 60729392
 P 6900 2950
@@
 	7300 2950 7300 3050
 $Comp
-L 1825910-6:1825910-6 SW8
+L macropad-v2_0_1-rescue:1825910-6-1825910-6 SW8
 U 1 1 6072FEF7
 P 3600 6750
@@
 Wire Wire Line
 	3600 3250 4650 3250
-Wire Wire Line
-	6250 3750 6250 3550
-Wire Wire Line
-	6250 3550 6050 3550
-Wire Wire Line
-	6250 3750 6650 3750
-Wire Wire Line
-	6050 3650 6300 3650
-Wire Wire Line
-	6300 3650 6300 3550
-Wire Wire Line
-	6300 3550 6650 3550
+Text GLabel 5700 5100 0    50   Input ~ 0
+Encoder_A
+Text GLabel 5700 5300 0    50   Input ~ 0
+Encoder_B
+Text GLabel 4650 3450 0    50   Input ~ 0
+Encoder_A
+Text GLabel 4650 3550 0    50   Input ~ 0
+Encoder_B
+Text GLabel 4650 3850 0    50   Input ~ 0
+Row_1
+Text GLabel 4650 3750 0    50   Input ~ 0
+Row_0
+NoConn ~ 4650 3650
+NoConn ~ 4650 3350
 $EndSCHEMATC
